File: JETT.kicad_sch (KiCad schematic)
At the start: 2 parts

Commit message: Add files via upload
Parts:
- added H1, H2, H3, H4: MountingHole, MountingHole:MountingHole_2.2mm_M2, symbol Mechanical:MountingHole
- B1, B2: footprint Panelization:MouseBite-Slot_2.0x2.0mm_outset_D0.5mm_P0.85mm_3h -> Panelization.pretty-master:mouse-bite-2mm-slot
