File: Right.kicad_sch (KiCad schematic)
At the start: 58 parts, among them J4 AudioJack4, SW15 SW_Push, SW20 SW_Push, SW23 SW_Push, SW25 SW_Push, SW26 SW_Push, SW27 SW_Push, SW28 SW_Push, SW29 SW_Push, SW31 SW_Push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

Commit message: Add files via upload
Parts:
- A2: footprint Module:RaspberryPi_Pico_Common_Unspecified -> Module:RaspberryPi_Pico_Common_SMD
Changed lines of the file:
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@@
 			)
 		)
-		(property "Footprint" "Module:RaspberryPi_Pico_Common_Unspecified"
+		(property "Footprint" "Module:RaspberryPi_Pico_Common_SMD"
 			(at 48.26 134.62 0)
 			(hide yes)
