File: JETT.kicad_pcb (KiCad board)
At the start: 2 copper layers, 290.1 x 128 mm, 120 parts, among them J3 AudioJack4, J4 AudioJack4, SW1 SW_Push, SW10 SW_Push, SW11 SW_Push, SW12 SW_Push, SW13 SW_Push, SW14 SW_Push, SW15 SW_Push, SW16 SW_Push, SW17 SW_Push, SW18 SW_Push, SW19 SW_Push, SW2 SW_Push, SW20 SW_Push, SW21 SW_Push, SW22 SW_Push, SW23 SW_Push, SW24 SW_Push, SW25 SW_Push, SW26 SW_Push, SW27 SW_Push, SW28 SW_Push, SW29 SW_Push, SW3 SW_Push, SW30 SW_Push, SW31 SW_Push, SW32 SW_Push, SW33 SW_Push, SW34 SW_Push, SW35 SW_Push, SW36 SW_Push, SW37 SW_Push, SW38 SW_Push, SW39 SW_Push, SW4 SW_Push, SW40 SW_Push, SW41 SW_Push, SW42 SW_Push, SW43 SW_Push, SW44 SW_Push, SW45 SW_Push, SW46 SW_Push, SW47 SW_Push, SW48 SW_Push, SW49 SW_Push, SW5 SW_Push, SW50 SW_Push, SW51 SW_Push, SW52 SW_Push, SW53 SW_Push, SW54 SW_Push, SW56 SW_Push, SW57 SW_Push, SW6 SW_Push, SW7 SW_Push, SW8 SW_Push, SW9 SW_Push

Commit message: Add files via upload
Parts:
- added H1: MountingHole, MountingHole:MountingHole_2.2mm_M2, F.Cu at (100.0, 139.8)
- added H2: MountingHole, MountingHole:MountingHole_2.2mm_M2, F.Cu at (128.0, 161.5)
- added H3: MountingHole, MountingHole:MountingHole_2.2mm_M2, F.Cu at (345.8, 139.8)
- added H4: MountingHole, MountingHole:MountingHole_2.2mm_M2, F.Cu at (317.8, 161.6)
- A1, A2: footprint Module:RaspberryPi_Pico_Common_Unspecified -> Module:RaspberryPi_Pico_Common_SMD
- moved J4 0.56 mm to (84.6, 144.0)
Routing:
- net /Left/COL_6: track 101.9 -> 88.9 mm
- net GND: track 39.3 -> 43.6 mm, vias 1 -> 2
- net /Left/ROW_3: track 148.0 -> 150.0 mm, vias 6 -> 7
- net /Left/ROW_4: track 159.4 -> 160.3 mm, vias 6 -> 7
- net /Right/COL_3: track 192.2 -> 191.4 mm, vias 2 -> 3
- net /Left/COL_1: track 173.3 -> 172.5 mm, vias 4 -> 5
- net /Left/COL_4: track 170.1 -> 169.3 mm, vias 2 -> 3
- net /Right/COL_2: track 168.4 -> 167.6 mm, vias 2 -> 3
- net /Left/ROW_2: track 141.4 -> 140.7 mm, vias 6 -> 7
- net /Left/ROW_1: track 156.1 -> 155.3 mm, vias 7 -> 8
- net /Right/COL_1: track 178.4 -> 177.8 mm, vias 0 -> 1
- net /Right/COL_5: track 153.6 -> 153.2 mm, vias 0 -> 1
- net /Right/ROW_5: track 108.3 -> 108.6 mm, vias 4 -> 5
- net /Right/COL_6: track 109.2 -> 109.4 mm, vias 0 -> 1
Other:
- outline, holes or cut-outs redrawn

Commit message: Add files via upload
Connections:
- A1 pad 1: /Left/COL_6 -> Net-(A1-GPIO0)
- A1 pad 21: Net-(A1-GPIO16) -> /Left/COL_6
- J3 pad R1: Net-(A1-GPIO16) -> Net-(A1-GPIO0)
Routing:
- net Net-(A1-GPIO0): track 0.00 -> 71.6 mm, vias 0 -> 2
- net /Left/COL_6: track 88.9 -> 119.2 mm, vias 0 -> 1
- net Net-(A1-GPIO16): track 16.1 -> 0.00 mm
Changed lines of the file:
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@@
 		(sheetname "/Right/")
 		(sheetfile "Right.kicad_sch")
+		(units
+			(unit
+				(name "A")
+				(pins "S" "R2" "R1" "T")
+			)
+		)
 		(attr smd)
 		(duplicate_pad_numbers_are_jumpers no)
@@
 			(size 1.6 0.8)
 			(layers "F.Cu" "F.Mask")
-			(net "/Left/COL_6")
+			(net "Net-(A1-GPIO0)")
 			(pinfunction "GPIO0_1")
 			(pintype "bidirectional")
@@
 			(layers "F.Cu" "F.Mask")
 			(roundrect_rratio 0.5)
-			(net "Net-(A1-GPIO16)")
+			(net "/Left/COL_6")
 			(pinfunction "GPIO16_21")
 			(pintype "bidirectional")
@@
 		(sheetname "/Left/")
 		(sheetfile "Left.kicad_sch")
+		(units
+			(unit
+				(name "A")
+				(pins "S" "R2" "R1" "T")
+			)
+		)
 		(attr smd)
 		(duplicate_pad_numbers_are_jumpers no)
@@
 			(size 1.2 2.5)
 			(layers "F.Cu" "F.Mask" "F.Paste")
-			(net "Net-(A1-GPIO16)")
+			(net "Net-(A1-GPIO0)")
 			(pintype "passive")
 		)
@@
 	)
 	(segment
+		(start 363.7 134.67)
+		(end 363.7 136.8)
+		(width 0.2)
+		(layer "F.Cu")
+		(net "/Left/COL_6")
+	)
+	(segment
 		(start 336.11 110.9)
 		(end 336.11 90.9)
@@
 	)
 	(segment
+		(start 365.26 133.11)
+		(end 363.7 134.67)
+		(width 0.2)
+		(layer "F.Cu")
+		(net "/Left/COL_6")
+	)
+	(segment
 		(start 336.11 130.9)
 		(end 336.11 110.9)
@@
 		(net "/Left/COL_6")
 	)
+	(via
+		(at 363.7 136.8)
+		(size 0.6)
+		(drill 0.3)
+		(layers "F.Cu" "B.Cu")
+		(net "/Left/COL_6")
+	)
+	(segment
+		(start 363.7 136.8)
+		(end 349.6 150.9)
+		(width 0.2)
+		(layer "B.Cu")
+		(net "/Left/COL_6")
+	)
+	(segment
+		(start 349.6 150.9)
+		(end 343.519189 150.9)
+		(width 0.2)
+		(layer "B.Cu")
+		(net "/Left/COL_6")
+	)
 	(segment
 		(start 336.11 150.9)
@@
 	)
 	(segment
-		(start 365.26 133.11)
-		(end 360.745 137.625)
+		(start 345.88 84.85)
+		(end 351.46 90.43)
+		(width 0.2)
+		(layer "F.Cu")
+		(net "Net-(A1-GPIO0)")
+	)
+	(segment
+		(start 351.46 90.43)
+		(end 351.46 113.86)
 		(width 0.2)
 		(layer "F.Cu")
-		(net "Net-(A1-GPIO16)")
+		(net "Net-(A1-GPIO0)")
 	)
 	(segment
-		(start 360.745 137.625)
+		(start 360.8 145)
+		(end 360.745 145.055)
+		(width 0.2)
+		(layer "F.Cu")
+		(net "Net-(A1-GPIO0)")
+	)
+	(segment
+		(start 351.46 113.86)
+		(end 362.6 125)
+		(width 0.2)
+		(layer "F.Cu")
+		(net "Net-(A1-GPIO0)")
+	)
+	(segment
+		(start 360.745 145.055)
 		(end 360.745 147.3)
 		(width 0.2)
 		(layer "F.Cu")
-		(net "Net-(A1-GPIO16)")
+		(net "Net-(A1-GPIO0)")
+	)
+	(via
+		(at 360.8 145)
+		(size 0.6)
+		(drill 0.3)
+		(layers "F.Cu" "B.Cu")
+		(net "Net-(A1-GPIO0)")
+	)
+	(via
+		(at 362.6 125)
+		(size 0.6)
+		(drill 0.3)
+		(layers "F.Cu" "B.Cu")
+		(net "Net-(A1-GPIO0)")
+	)
+	(segment
+		(start 364.3 126.7)
+		(end 364.3 141.5)
+		(width 0.2)
+		(layer "B.Cu")
+		(net "Net-(A1-GPIO0)")
+	)
+	(segment
+		(start 362.6 125)
+		(end 364.3 126.7)
+		(width 0.2)
+		(layer "B.Cu")
+		(net "Net-(A1-GPIO0)")
+	)
+	(segment
+		(start 364.3 141.5)
+		(end 360.8 145)
+		(width 0.2)
+		(layer "B.Cu")
+		(net "Net-(A1-GPIO0)")
 	)
 	(embedded_fonts no)
