File: Left.kicad_sch (KiCad schematic)
At the start: 58 parts, among them J3 AudioJack4, SW1 SW_Push, SW10 SW_Push, SW11 SW_Push, SW12 SW_Push, SW13 SW_Push, SW14 SW_Push, SW16 SW_Push, SW17 SW_Push, SW18 SW_Push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

Commit message: Add files via upload
Parts:
- A1: footprint Module:RaspberryPi_Pico_Common_Unspecified -> Module:RaspberryPi_Pico_Common_SMD
Changed lines of the file:
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@@
 			)
 		)
-		(property "Footprint" "Module:RaspberryPi_Pico_Common_Unspecified"
+		(property "Footprint" "Module:RaspberryPi_Pico_Common_SMD"
 			(at 53.34 138.43 0)
 			(hide yes)

Commit message: Add files via upload
Connections:
- net COL_6: now also A1.21 (GPIO16); no longer A1.1 (GPIO0)
- net at J3.R1: now also A1.1 (GPIO0); no longer A1.21 (GPIO16)
Changed lines of the file:
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@@
+	(wire
+		(pts
+			(xy 83.82 78.74) (xy 76.2 78.74)
+		)
+		(stroke
+			(width 0)
+			(type default)
+		)
+	)
 	(wire
 		(pts
@@
 	(wire
 		(pts
+			(xy 30.48 76.2) (xy 29.21 76.2)
+		)
+		(stroke
+			(width 0)
+			(type default)
+		)
+	)
+	(wire
+		(pts
 			(xy 130.81 40.64) (xy 130.81 63.5)
 		)
@@
 	(wire
 		(pts
+			(xy 29.21 76.2) (xy 29.21 50.8)
+		)
+		(stroke
+			(width 0)
+			(type default)
+		)
+	)
+	(wire
+		(pts
 			(xy 186.69 88.9) (xy 186.69 111.76)
 		)
@@
 	(wire
 		(pts
+			(xy 29.21 50.8) (xy 60.96 50.8)
+		)
+		(stroke
+			(width 0)
+			(type default)
+		)
+	)
+	(wire
+		(pts
 			(xy 114.3 63.5) (xy 114.3 66.04)
 		)
@@
 	(wire
 		(pts
-			(xy 76.2 54.61) (xy 76.2 78.74)
-		)
-		(stroke
-			(width 0)
-			(type default)
-		)
-	)
-	(wire
-		(pts
 			(xy 242.57 40.64) (xy 242.57 63.5)
 		)
@@
 	(wire
 		(pts
-			(xy 60.96 54.61) (xy 76.2 54.61)
-		)
-		(stroke
-			(width 0)
-			(type default)
-		)
-	)
-	(wire
-		(pts
-			(xy 22.86 76.2) (xy 30.48 76.2)
-		)
-		(stroke
-			(width 0)
-			(type default)
-		)
-	)
-	(wire
-		(pts
 			(xy 252.73 73.66) (xy 273.05 73.66)
 		)
@@
 	(wire
 		(pts
-			(xy 60.96 45.72) (xy 60.96 54.61)
+			(xy 60.96 45.72) (xy 60.96 50.8)
 		)
 		(stroke
@@
 		)
 	)
+	(label "COL_6"
+		(at 83.82 78.74 180)
+		(effects
+			(font
+				(size 1.27 1.27)
+			)
+			(justify right bottom)
+		)
+	)
 	(label "ROW_4"
 		(at 22.86 99.06 0)
@@
 		)
 	)
-	(label "COL_6"
-		(at 22.86 76.2 0)
-		(effects
-			(font
-				(size 1.27 1.27)
-			)
-			(justify left bottom)
-		)
-	)
